File: kicad/amplificador.sch (KiCad schematic (older format))
At the start: 55 parts, among them Q1 BC557, Q10 BC547, Q11 BC547, Q12 BC557, Q13 BC547, Q14 BC557, Q15 TIP41C, Q16 TIP41C, Q17 TIP42C, Q18 TIP42C, Q2 BC547, Q3 BC557, Q4 BC547, Q5 BC557, Q6 BC557, Q7 BC547, Q8 BC557, Q9 BC547

Commit message: Inicio del ruteo
Parts:
- C1, C2, C4: footprint (none) -> Capacitor_SMD:CP_Elec_3x5.3
- C3: footprint (none) -> Capacitor_THT:CP_Radial_D7.5mm_P2.50mm
- C5: value C -> 100p; footprint (none) -> Capacitor_SMD:CP_Elec_3x5.3
- C6: value C -> 22n; footprint (none) -> Capacitor_SMD:CP_Elec_3x5.3
- Q1, Q10, Q11, Q12, Q13, Q14, Q2, Q3, Q4, Q5, Q6, Q7, Q8, Q9: footprint Package_TO_SOT_THT:TO-92_Inline -> Package_TO_SOT_THT:TO-92
- R17: value 1.6k -> 1.2k
Changed lines of the file:
@@
 F 0 "C3" H 4315 4446 50  0000 L CNN
 F 1 "1000u" H 4315 4355 50  0000 L CNN
-F 2 "" H 4238 4250 50  0001 C CNN
+F 2 "Capacitor_THT:CP_Radial_D7.5mm_P2.50mm" H 4238 4250 50  0001 C CNN
 F 3 "~" H 4200 4400 50  0001 C CNN
 	1    4200 4400
@@
 F 0 "C4" V 4498 2750 50  0000 C CNN
 F 1 "47u" V 4589 2750 50  0000 C CNN
-F 2 "" H 4788 2600 50  0001 C CNN
+F 2 "Capacitor_SMD:CP_Elec_3x5.3" H 4788 2600 50  0001 C CNN
 F 3 "~" H 4750 2750 50  0001 C CNN
 	1    4750 2750
@@
 F 0 "C2" H 3285 1654 50  0000 R CNN
 F 1 "47u" H 3285 1745 50  0000 R CNN
-F 2 "" H 3438 1550 50  0001 C CNN
+F 2 "Capacitor_SMD:CP_Elec_3x5.3" H 3438 1550 50  0001 C CNN
 F 3 "~" H 3400 1700 50  0001 C CNN
 	1    3400 1700
@@
 P 5300 4700
 F 0 "C5" V 5048 4700 50  0000 C CNN
-F 1 "C" V 5139 4700 50  0000 C CNN
-F 2 "" H 5338 4550 50  0001 C CNN
+F 1 "100p" V 5139 4700 50  0000 C CNN
+F 2 "Capacitor_SMD:CP_Elec_3x5.3" H 5338 4550 50  0001 C CNN
 F 3 "~" H 5300 4700 50  0001 C CNN
 	1    5300 4700
@@
 F 0 "C1" V 948 3850 50  0000 C CNN
 F 1 "47u" V 1039 3850 50  0000 C CNN
-F 2 "" H 1238 3700 50  0001 C CNN
+F 2 "Capacitor_SMD:CP_Elec_3x5.3" H 1238 3700 50  0001 C CNN
 F 3 "~" H 1200 3850 50  0001 C CNN
 	1    1200 3850
@@
 F 0 "Q9" H 6541 5796 50  0000 L CNN
 F 1 "BC547" H 6541 5705 50  0000 L CNN
-F 2 "Package_TO_SOT_THT:TO-92_Inline" H 6550 5675 50  0001 L CIN
+F 2 "Package_TO_SOT_THT:TO-92" H 6550 5675 50  0001 L CIN
 F 3 "http://www.fairchildsemi.com/ds/BC/BC547.pdf" H 6350 5750 50  0001 L CNN
 	1    6350 5750
@@
 F 0 "Q7" H 5441 5296 50  0000 L CNN
 F 1 "BC547" H 5441 5205 50  0000 L CNN
-F 2 "Package_TO_SOT_THT:TO-92_Inline" H 5450 5175 50  0001 L CIN
+F 2 "Package_TO_SOT_THT:TO-92" H 5450 5175 50  0001 L CIN
 F 3 "http://www.fairchildsemi.com/ds/BC/BC547.pdf" H 5250 5250 50  0001 L CNN
 	1    5250 5250
@@
 F 0 "Q4" H 3541 5396 50  0000 L CNN
 F 1 "BC547" H 3541 5305 50  0000 L CNN
-F 2 "Package_TO_SOT_THT:TO-92_Inline" H 3550 5275 50  0001 L CIN
+F 2 "Package_TO_SOT_THT:TO-92" H 3550 5275 50  0001 L CIN
 F 3 "http://www.fairchildsemi.com/ds/BC/BC547.pdf" H 3350 5350 50  0001 L CNN
 	1    3350 5350
@@
 F 0 "Q2" H 2491 5396 50  0000 L CNN
 F 1 "BC547" H 2491 5305 50  0000 L CNN
-F 2 "Package_TO_SOT_THT:TO-92_Inline" H 2500 5275 50  0001 L CIN
+F 2 "Package_TO_SOT_THT:TO-92" H 2500 5275 50  0001 L CIN
 F 3 "http://www.fairchildsemi.com/ds/BC/BC547.pdf" H 2300 5350 50  0001 L CNN
 	1    2300 5350
@@
 F 0 "Q1" H 2291 3896 50  0000 L CNN
 F 1 "BC557" H 2291 3805 50  0000 L CNN
-F 2 "Package_TO_SOT_THT:TO-92_Inline" H 2300 3775 50  0001 L CIN
+F 2 "Package_TO_SOT_THT:TO-92" H 2300 3775 50  0001 L CIN
 F 3 "http://www.fairchildsemi.com/ds/BC/BC557.pdf" H 2100 3850 50  0001 L CNN
 	1    2100 3850
@@
 F 0 "Q5" H 3741 3896 50  0000 L CNN
 F 1 "BC557" H 3741 3805 50  0000 L CNN
-F 2 "Package_TO_SOT_THT:TO-92_Inline" H 3750 3775 50  0001 L CIN
+F 2 "Package_TO_SOT_THT:TO-92" H 3750 3775 50  0001 L CIN
 F 3 "http://www.fairchildsemi.com/ds/BC/BC557.pdf" H 3550 3850 50  0001 L CNN
 	1    3550 3850
@@
 F 0 "Q3" H 3091 2204 50  0000 L CNN
 F 1 "BC557" H 3091 2295 50  0000 L CNN
-F 2 "Package_TO_SOT_THT:TO-92_Inline" H 3100 2175 50  0001 L CIN
+F 2 "Package_TO_SOT_THT:TO-92" H 3100 2175 50  0001 L CIN
 F 3 "http://www.fairchildsemi.com/ds/BC/BC557.pdf" H 2900 2250 50  0001 L CNN
 	1    2900 2250
@@
 F 0 "Q8" H 6541 2204 50  0000 L CNN
 F 1 "BC557" H 6541 2295 50  0000 L CNN
-F 2 "Package_TO_SOT_THT:TO-92_Inline" H 6550 2175 50  0001 L CIN
+F 2 "Package_TO_SOT_THT:TO-92" H 6550 2175 50  0001 L CIN
 F 3 "http://www.fairchildsemi.com/ds/BC/BC557.pdf" H 6350 2250 50  0001 L CNN
 	1    6350 2250
@@
 F 0 "Q6" H 5341 1804 50  0000 L CNN
 F 1 "BC557" H 5341 1895 50  0000 L CNN
-F 2 "Package_TO_SOT_THT:TO-92_Inline" H 5350 1775 50  0001 L CIN
+F 2 "Package_TO_SOT_THT:TO-92" H 5350 1775 50  0001 L CIN
 F 3 "http://www.fairchildsemi.com/ds/BC/BC557.pdf" H 5150 1850 50  0001 L CNN
 	1    5150 1850
@@
 F 0 "Q10" H 6541 3796 50  0000 L CNN
 F 1 "BC547" H 6541 3705 50  0000 L CNN
-F 2 "Package_TO_SOT_THT:TO-92_Inline" H 6550 3675 50  0001 L CIN
+F 2 "Package_TO_SOT_THT:TO-92" H 6550 3675 50  0001 L CIN
 F 3 "http://www.fairchildsemi.com/ds/BC/BC547.pdf" H 6350 3750 50  0001 L CNN
 	1    6350 3750
@@
 P 5800 4100
 F 0 "R17" H 5870 4146 50  0000 L CNN
-F 1 "1.6k" H 5870 4055 50  0000 L CNN
+F 1 "1.2k" H 5870 4055 50  0000 L CNN
 F 2 "Resistor_SMD:R_0805_2012Metric_Pad1.15x1.40mm_HandSolder" V 5730 4100 50  0001 C CNN
 F 3 "~" H 5800 4100 50  0001 C CNN
@@
 P 6950 3700
 F 0 "C6" V 6698 3700 50  0000 C CNN
-F 1 "C" V 6789 3700 50  0000 C CNN
-F 2 "" H 6988 3550 50  0001 C CNN
+F 1 "22n" V 6789 3700 50  0000 C CNN
+F 2 "Capacitor_SMD:CP_Elec_3x5.3" H 6988 3550 50  0001 C CNN
 F 3 "~" H 6950 3700 50  0001 C CNN
 	1    6950 3700
@@
 F 0 "Q11" H 8041 2046 50  0000 L CNN
 F 1 "BC547" H 8041 1955 50  0000 L CNN
-F 2 "Package_TO_SOT_THT:TO-92_Inline" H 8050 1925 50  0001 L CIN
+F 2 "Package_TO_SOT_THT:TO-92" H 8050 1925 50  0001 L CIN
 F 3 "http://www.fairchildsemi.com/ds/BC/BC547.pdf" H 7850 2000 50  0001 L CNN
 	1    7850 2000
@@
 F 0 "Q13" H 8541 3346 50  0000 L CNN
 F 1 "BC547" H 8541 3255 50  0000 L CNN
-F 2 "Package_TO_SOT_THT:TO-92_Inline" H 8550 3225 50  0001 L CIN
+F 2 "Package_TO_SOT_THT:TO-92" H 8550 3225 50  0001 L CIN
 F 3 "http://www.fairchildsemi.com/ds/BC/BC547.pdf" H 8350 3300 50  0001 L CNN
 	1    8350 3300
@@
 F 0 "Q14" H 8541 4654 50  0000 L CNN
 F 1 "BC557" H 8541 4745 50  0000 L CNN
-F 2 "Package_TO_SOT_THT:TO-92_Inline" H 8550 4625 50  0001 L CIN
+F 2 "Package_TO_SOT_THT:TO-92" H 8550 4625 50  0001 L CIN
 F 3 "http://www.fairchildsemi.com/ds/BC/BC557.pdf" H 8350 4700 50  0001 L CNN
 	1    8350 4700
@@
 F 0 "Q12" H 8041 5704 50  0000 L CNN
 F 1 "BC557" H 8041 5795 50  0000 L CNN
-F 2 "Package_TO_SOT_THT:TO-92_Inline" H 8050 5675 50  0001 L CIN
+F 2 "Package_TO_SOT_THT:TO-92" H 8050 5675 50  0001 L CIN
 F 3 "http://www.fairchildsemi.com/ds/BC/BC557.pdf" H 7850 5750 50  0001 L CNN
 	1    7850 5750
