File: kicad/_autosave-amplificador.sch (KiCad schematic (older format))
At the start: 77 parts, among them J1 Screw_Terminal_01x01, J10 Conn_01x01_Male, J11 Conn_01x01_Male, J12 Conn_01x01_Male, J13 Conn_01x01_Male, J14 Conn_01x01_Male, J15 Conn_01x01_Male, J16 Screw_Terminal_01x01, J17 Screw_Terminal_01x01, J2 Conn_01x01_Male, J3 Conn_01x01_Male, J4 Conn_01x01_Male, J5 Conn_01x01_Male, J6 Conn_01x01_Male, J7 Screw_Terminal_01x01, J8 Screw_Terminal_01x01, J9 Conn_01x01_Male, Q1 MPSA92, Q10 MPSA42, Q11 BD135, Q12 BD136, Q13 BD135, Q14 BD136, Q15 2SD1047, Q16 2SD1047, Q17 2SB817, Q18 2SB817, Q2 MPSA42, Q3 MPSA92, Q4 MPSA42, Q5 MPSA92, Q6 MPSA92, Q7 MPSA42, Q8 MPSA92, Q9 MPSA42, U1 LM385D-1.2, U2 LM385D-1.2

Commit message: carpeta kicad con esquematico con todos los encapsulados correctos, jumpers, pines de alimentacion y medicon. pcb a medio hacer
Parts:
- C1: footprint Capacitor_THT:C_Disc_D16.0mm_W5.0mm_P7.50mm -> Capacitor_THT:C_Disc_D10.0mm_W2.5mm_P5.00mm
- J1, J16, J17, J7, J8: footprint Connector_Wire:SolderWirePad_1x01_Drill2mm -> Connector_Wire:SolderWirePad_1x01_Drill0.8mm
- J10, J11, J12, J13, J14, J15, J2, J3, J4, J5, J6, J9: footprint Connector_Wire:SolderWirePad_1x01_Drill2mm -> Connector_Pin:Pin_D0.7mm_L6.5mm_W1.8mm_FlatFork
Changed lines of the file:
@@
 F 0 "C1" V 948 3850 50  0000 C CNN
 F 1 "10u" V 1039 3850 50  0000 C CNN
-F 2 "Capacitor_THT:C_Disc_D16.0mm_W5.0mm_P7.50mm" H 1238 3700 50  0001 C CNN
+F 2 "Capacitor_THT:C_Disc_D10.0mm_W2.5mm_P5.00mm" H 1238 3700 50  0001 C CNN
 F 3 "~" H 1200 3850 50  0001 C CNN
 	1    1200 3850
@@
 F 0 "J8" V 5014 712 50  0000 R CNN
 F 1 "Screw_Terminal_01x01" V 4923 712 50  0000 R CNN
-F 2 "Connector_Wire:SolderWirePad_1x01_Drill2mm" H 5050 800 50  0001 C CNN
+F 2 "Connector_Wire:SolderWirePad_1x01_Drill0.8mm" H 5050 800 50  0001 C CNN
 F 3 "~" H 5050 800 50  0001 C CNN
 	1    5050 800
@@
 F 0 "J7" V 4472 7680 50  0000 L CNN
 F 1 "Screw_Terminal_01x01" V 4563 7680 50  0000 L CNN
-F 2 "Connector_Wire:SolderWirePad_1x01_Drill2mm" H 4600 7600 50  0001 C CNN
+F 2 "Connector_Wire:SolderWirePad_1x01_Drill0.8mm" H 4600 7600 50  0001 C CNN
 F 3 "~" H 4600 7600 50  0001 C CNN
 	1    4600 7600
@@
 F 0 "J1" H 768 3625 50  0000 C CNN
 F 1 "Screw_Terminal_01x01" H 768 3716 50  0000 C CNN
-F 2 "Connector_Wire:SolderWirePad_1x01_Drill2mm" H 850 3850 50  0001 C CNN
+F 2 "Connector_Wire:SolderWirePad_1x01_Drill0.8mm" H 850 3850 50  0001 C CNN
 F 3 "~" H 850 3850 50  0001 C CNN
 	1    850  3850
@@
 F 0 "J16" H 10130 4842 50  0000 L CNN
 F 1 "Screw_Terminal_01x01" H 10130 4751 50  0000 L CNN
-F 2 "Connector_Wire:SolderWirePad_1x01_Drill2mm" H 10050 4800 50  0001 C CNN
+F 2 "Connector_Wire:SolderWirePad_1x01_Drill0.8mm" H 10050 4800 50  0001 C CNN
 F 3 "~" H 10050 4800 50  0001 C CNN
 	1    10050 4800
@@
 F 0 "J17" H 10180 2792 50  0000 L CNN
 F 1 "Screw_Terminal_01x01" H 10180 2701 50  0000 L CNN
-F 2 "Connector_Wire:SolderWirePad_1x01_Drill2mm" H 10100 2750 50  0001 C CNN
+F 2 "Connector_Wire:SolderWirePad_1x01_Drill0.8mm" H 10100 2750 50  0001 C CNN
 F 3 "~" H 10100 2750 50  0001 C CNN
 	1    10100 2750
@@
 F 0 "J3" H 2108 6081 50  0000 C CNN
 F 1 "Conn_01x01_Male" H 2108 5990 50  0000 C CNN
-F 2 "Connector_Wire:SolderWirePad_1x01_Drill2mm" H 2000 5900 50  0001 C CNN
+F 2 "Connector_Pin:Pin_D0.7mm_L6.5mm_W1.8mm_FlatFork" H 2000 5900 50  0001 C CNN
 F 3 "~" H 2000 5900 50  0001 C CNN
 	1    2000 5900
@@
 F 0 "J6" H 3358 6081 50  0000 C CNN
 F 1 "Conn_01x01_Male" H 3358 5990 50  0000 C CNN
-F 2 "Connector_Wire:SolderWirePad_1x01_Drill2mm" H 3250 5900 50  0001 C CNN
+F 2 "Connector_Pin:Pin_D0.7mm_L6.5mm_W1.8mm_FlatFork" H 3250 5900 50  0001 C CNN
 F 3 "~" H 3250 5900 50  0001 C CNN
 	1    3250 5900
@@
 F 0 "J4" H 2708 2181 50  0000 C CNN
 F 1 "Conn_01x01_Male" H 2708 2090 50  0000 C CNN
-F 2 "Connector_Wire:SolderWirePad_1x01_Drill2mm" H 2600 2000 50  0001 C CNN
+F 2 "Connector_Pin:Pin_D0.7mm_L6.5mm_W1.8mm_FlatFork" H 2600 2000 50  0001 C CNN
 F 3 "~" H 2600 2000 50  0001 C CNN
 	1    2600 2000
@@
 F 0 "J2" H 2108 3781 50  0000 C CNN
 F 1 "Conn_01x01_Male" H 2108 3690 50  0000 C CNN
-F 2 "Connector_Wire:SolderWirePad_1x01_Drill2mm" H 2000 3600 50  0001 C CNN
+F 2 "Connector_Pin:Pin_D0.7mm_L6.5mm_W1.8mm_FlatFork" H 2000 3600 50  0001 C CNN
 F 3 "~" H 2000 3600 50  0001 C CNN
 	1    2000 3600
@@
 F 0 "J5" H 3358 3781 50  0000 C CNN
 F 1 "Conn_01x01_Male" H 3358 3690 50  0000 C CNN
-F 2 "Connector_Wire:SolderWirePad_1x01_Drill2mm" H 3250 3600 50  0001 C CNN
+F 2 "Connector_Pin:Pin_D0.7mm_L6.5mm_W1.8mm_FlatFork" H 3250 3600 50  0001 C CNN
 F 3 "~" H 3250 3600 50  0001 C CNN
 	1    3250 3600
@@
 F 0 "J9" H 6358 1931 50  0000 C CNN
 F 1 "Conn_01x01_Male" H 6358 1840 50  0000 C CNN
-F 2 "Connector_Wire:SolderWirePad_1x01_Drill2mm" H 6250 1750 50  0001 C CNN
+F 2 "Connector_Pin:Pin_D0.7mm_L6.5mm_W1.8mm_FlatFork" H 6250 1750 50  0001 C CNN
 F 3 "~" H 6250 1750 50  0001 C CNN
 	1    6250 1750
@@
 F 0 "J14" H 9158 3881 50  0000 C CNN
 F 1 "Conn_01x01_Male" H 9158 3790 50  0000 C CNN
-F 2 "Connector_Wire:SolderWirePad_1x01_Drill2mm" H 9050 3700 50  0001 C CNN
+F 2 "Connector_Pin:Pin_D0.7mm_L6.5mm_W1.8mm_FlatFork" H 9050 3700 50  0001 C CNN
 F 3 "~" H 9050 3700 50  0001 C CNN
 	1    9050 3700
@@
 F 0 "J15" H 9158 4531 50  0000 C CNN
 F 1 "Conn_01x01_Male" H 9158 4440 50  0000 C CNN
-F 2 "Connector_Wire:SolderWirePad_1x01_Drill2mm" H 9050 4350 50  0001 C CNN
+F 2 "Connector_Pin:Pin_D0.7mm_L6.5mm_W1.8mm_FlatFork" H 9050 4350 50  0001 C CNN
 F 3 "~" H 9050 4350 50  0001 C CNN
 	1    9050 4350
@@
 F 0 "J10" V 7962 3144 50  0000 L CNN
 F 1 "Conn_01x01_Male" V 8053 3144 50  0000 L CNN
-F 2 "Connector_Wire:SolderWirePad_1x01_Drill2mm" H 7900 3100 50  0001 C CNN
+F 2 "Connector_Pin:Pin_D0.7mm_L6.5mm_W1.8mm_FlatFork" H 7900 3100 50  0001 C CNN
 F 3 "~" H 7900 3100 50  0001 C CNN
 	1    7900 3100
@@
 F 0 "J11" V 7962 4544 50  0000 L CNN
 F 1 "Conn_01x01_Male" V 8053 4544 50  0000 L CNN
-F 2 "Connector_Wire:SolderWirePad_1x01_Drill2mm" H 7900 4500 50  0001 C CNN
+F 2 "Connector_Pin:Pin_D0.7mm_L6.5mm_W1.8mm_FlatFork" H 7900 4500 50  0001 C CNN
 F 3 "~" H 7900 4500 50  0001 C CNN
 	1    7900 4500
@@
 F 0 "J13" H 8358 4531 50  0000 C CNN
 F 1 "Conn_01x01_Male" H 8358 4440 50  0000 C CNN
-F 2 "Connector_Wire:SolderWirePad_1x01_Drill2mm" H 8250 4350 50  0001 C CNN
+F 2 "Connector_Pin:Pin_D0.7mm_L6.5mm_W1.8mm_FlatFork" H 8250 4350 50  0001 C CNN
 F 3 "~" H 8250 4350 50  0001 C CNN
 	1    8250 4350
@@
 F 0 "J12" H 8358 3831 50  0000 C CNN
 F 1 "Conn_01x01_Male" H 8358 3740 50  0000 C CNN
-F 2 "Connector_Wire:SolderWirePad_1x01_Drill2mm" H 8250 3650 50  0001 C CNN
+F 2 "Connector_Pin:Pin_D0.7mm_L6.5mm_W1.8mm_FlatFork" H 8250 3650 50  0001 C CNN
 F 3 "~" H 8250 3650 50  0001 C CNN
 	1    8250 3650
