File: kicad/_autosave-amplificador.kicad_pcb (KiCad board)
At the start: 2 copper layers, 79 parts, among them J1 Screw_Terminal_01x01, J10 Conn_01x01_Male, J11 Conn_01x01_Male, J12 Conn_01x01_Male, J13 Conn_01x01_Male, J16 Screw_Terminal_01x01, J17 Screw_Terminal_01x01, J18 Conn_01x01_Male, J19 Conn_01x01_Male, J2 Conn_01x01_Male, J3 Conn_01x01_Male, J4 Conn_01x01_Male, J5 Conn_01x01_Male, J6 Conn_01x01_Male, J7 Screw_Terminal_01x01, J8 Screw_Terminal_01x01, J9 Conn_01x01_Male, Q1 MPSA92, Q10 MPSA42, Q11 BD135, Q12 BD136, Q13 BD135, Q14 BD136, Q15 2SD1047, Q16 2SD1047, Q17 2SB817, Q18 2SB817, Q2 MPSA42, Q3 MPSA92, Q4 MPSA42, Q5 MPSA92, Q6 MPSA92, Q7 MPSA42, Q8 MPSA92, Q9 MPSA42, U1 LM385D-1.2, U2 LM385D-1.2

Commit message: intento de optimización de pcb: seguramente haya que volver a la versión anterior y tirar una via para la realimentación...
Parts:
- moved J17 176.0 mm to (276.9, 154.9), turned to 270 degrees
- moved Q15 163.1 mm to (276.9, 121.9), turned to 90 degrees
- moved D6 157.5 mm to (276.9, 132.1), turned to 270 degrees
- moved Q16 139.2 mm to (276.9, 99.8), turned to 90 degrees
- moved C4 122.2 mm to (171.4, 63.5), turned to 90 degrees
- moved R24 121.9 mm to (270.5, 90.2), turned to 180 degrees
- moved Q17 113.7 mm to (276.9, 71.1), turned to 90 degrees
- moved R10 113.5 mm to (167.4, 69.8), turned to 180 degrees
- moved Q6 113.4 mm to (189.2, 71.1), turned to 180 degrees
- moved R9 113.2 mm to (175.0, 69.8), turned to 180 degrees
- moved R6 112.1 mm to (232.4, 66.0), turned to 270 degrees
- moved J6 107.8 mm to (232.4, 62.2), turned to 0 degrees
- moved R15 107.1 mm to (182.9, 45.5), turned to 90 degrees
- moved R2 103.6 mm to (221.0, 66.0), turned to 90 degrees
- moved Q18 102.9 mm to (278.1, 49.5), turned to 90 degrees
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