File: smps/kicad/negativa/negativa/negativa.sch (KiCad schematic (older format))
At the start: 18 parts, among them J1 Conn_01x01_Female, J2 Conn_01x01_Female, J3 Conn_01x01_Female, J4 Conn_01x01_Female, Q1 2N3906, U1 LM2577T-ADJ

Commit message: varias cosas, layouts de fuentes terminados, calculo de componentes completo
Parts:
- C1: footprint Capacitor_THT:CP_Radial_D16.0mm_P7.50mm -> Capacitor_SMD:C_1206_3216Metric_Pad1.33x1.80mm_HandSolder
- C2: footprint Capacitor_THT:CP_Radial_D16.0mm_P7.50mm -> Capacitor_THT:CP_Radial_D8.0mm_P3.50mm
- C3: value 100u -> 0.22u; footprint Capacitor_THT:CP_Radial_D16.0mm_P7.50mm -> Capacitor_SMD:C_1206_3216Metric_Pad1.33x1.80mm_HandSolder
- R3: value 4.12k -> 4.3k
Changed lines of the file:
@@
 P 6350 5750
 F 0 "R3" H 6420 5796 50  0000 L CNN
-F 1 "4.12k" H 6420 5705 50  0000 L CNN
+F 1 "4.3k" H 6420 5705 50  0000 L CNN
 F 2 "Resistor_SMD:R_1206_3216Metric_Pad1.30x1.75mm_HandSolder" V 6280 5750 50  0001 C CNN
 F 3 "~" H 6350 5750 50  0001 C CNN
@@
 F 0 "C1" H 3215 4246 50  0000 L CNN
 F 1 "0.22u" H 3215 4155 50  0000 L CNN
-F 2 "Capacitor_THT:CP_Radial_D16.0mm_P7.50mm" H 3138 4050 50  0001 C CNN
+F 2 "Capacitor_SMD:C_1206_3216Metric_Pad1.33x1.80mm_HandSolder" H 3138 4050 50  0001 C CNN
 F 3 "~" H 3100 4200 50  0001 C CNN
 	1    3100 4200
@@
 F 0 "C2" H 4482 2754 50  0000 R CNN
 F 1 "100u" H 4482 2845 50  0000 R CNN
-F 2 "Capacitor_THT:CP_Radial_D16.0mm_P7.50mm" H 4638 2650 50  0001 C CNN
+F 2 "Capacitor_THT:CP_Radial_D8.0mm_P3.50mm" H 4638 2650 50  0001 C CNN
 F 3 "~" H 4600 2800 50  0001 C CNN
 	1    4600 2800
@@
 P 5050 2800
 F 0 "C3" H 4932 2754 50  0000 R CNN
-F 1 "100u" H 4932 2845 50  0000 R CNN
-F 2 "Capacitor_THT:CP_Radial_D16.0mm_P7.50mm" H 5088 2650 50  0001 C CNN
+F 1 "0.22u" H 4932 2845 50  0000 R CNN
+F 2 "Capacitor_SMD:C_1206_3216Metric_Pad1.33x1.80mm_HandSolder" H 5088 2650 50  0001 C CNN
 F 3 "~" H 5050 2800 50  0001 C CNN
 	1    5050 2800

Commit message: last minute commit
Parts:
- R3: value 4.3k -> 3.3k
Changed lines of the file:
@@
 P 6350 5750
 F 0 "R3" H 6420 5796 50  0000 L CNN
-F 1 "4.3k" H 6420 5705 50  0000 L CNN
+F 1 "3.3k" H 6420 5705 50  0000 L CNN
 F 2 "Resistor_SMD:R_1206_3216Metric_Pad1.30x1.75mm_HandSolder" V 6280 5750 50  0001 C CNN
 F 3 "~" H 6350 5750 50  0001 C CNN
